Commit message: grav comp works, no offset and hardware thresholds can be set

File: src/factr/factr_teleop/factr_teleop/urdf/factr_teleop_franka.urdf (robot description, URDF)
Before this commit: robot factr_teleop_franka, 8 links, 7 joints
Links:
- link link_2: mass 0.042 -> 0.037
- link link_4: mass 0.051 -> 0.046
- link link_5: mass 0.048 -> 0.043
- link link_6: mass 0.035 -> 0.03
- link link_7: mass 0.0 -> 0.046
